File: TS48_Right/LED+MATRIX.sch (KiCad schematic (older format))
At the start: 78 parts

Commit message: Layout changes
Connections:
- net +5V: now also MX1.3 (LED), MX10.3 (LED), MX11.3 (LED), MX12.3 (LED), MX13.3 (LED), MX14.3 (LED), MX15.3 (LED), MX16.3 (LED), MX17.3 (LED), MX18.3 (LED), MX19.3 (LED), MX2.3 (LED), MX20.3 (LED), MX21.3 (LED), MX22.3 (LED), MX23.3 (LED), MX24.3 (LED), MX25.3 (LED), MX26.3 (LED), MX27.3 (LED), MX28.3 (LED), MX29.3 (LED), MX3.3 (LED), MX30.4 (LEDGND), MX4.3 (LED), MX5.3 (LED), MX6.3 (LED), MX7.3 (LED), MX8.3 (LED), MX9.3 (LED); no longer MX1.4 (LEDGND), R5.1
- new net: MX1.4 (LEDGND), R5.1
Changed lines of the file:
@@
 	3375 2150 2450 2150
-Wire Wire Line
-	3000 1950 2450 1950
-Connection ~ 3000 1950
 Wire Wire Line
 	3150 1800 3150 1500
@@
 	8800 4200 8825 4200
 Wire Wire Line
-	8850 4925 9625 4925
-Wire Wire Line
-	9625 4925 9625 4150
-Wire Wire Line
-	9625 4150 9250 4150
-Connection ~ 9250 4150
-Wire Wire Line
 	8950 4825 8950 4050
 Wire Wire Line
@@
 Wire Wire Line
 	3150 3900 3150 4000
+Wire Wire Line
+	3100 1850 2500 1850
+Wire Wire Line
+	2500 1850 2500 1950
+Wire Wire Line
+	2500 1950 2450 1950
+Wire Wire Line
+	8875 4150 8875 4925
+Wire Wire Line
+	8875 4925 8850 4925
+Connection ~ 8875 4150
 $EndSCHEMATC
