File: TS48_Right/TS48_right.kicad_pcb (KiCad board)
At the start: 2 copper layers, 128.5 x 81 mm, 24 parts, among them SW0 SW_MX, SW1 SW_PUSH, SW10 SW_MX, SW11 SW_MX, SW12 SW_MX, SW13 SW_MX, SW14 SW_MX, SW15 SW_MX, SW16 SW_MX, SW17 SW_MX, SW18 SW_MX, SW19 SW_MX, SW2 SW_MX, SW20 SW_MX, SW21 SW_MX, SW22 SW_MX, SW23 SW_MX, SW3 SW_MX, SW4 SW_MX, SW5 SW_MX, SW6 SW_MX, SW7 SW_MX, SW8 SW_MX, SW9 SW_MX

Commit message: Layout changes
Parts:
- removed SW0, SW10, SW12, SW13, SW14, SW15, SW16, SW17, SW18, SW2, SW20, SW21, SW22, SW23, SW3, SW4, SW6, SW7, SW8, SW9: SW_MX, Cherry_MX_Matias_u1_NoSilk_Back
- removed SW11, SW19: SW_MX, Cherry_MX_Matias_u1.25_NoSilk_Back
- removed SW5: SW_MX, Cherry_MX_Matias_u1.5_NoSilk_Back
- added C1: 0.1uf, Capacitors_SMD:C_0805_HandSoldering, B.Cu at (204.7, 88.4)
- added C10: 0.1uF, Capacitors_SMD:C_0805_HandSoldering, B.Cu at (133.2, 83.9)
- added C11: 0.1uF, Capacitors_SMD:C_0805_HandSoldering, B.Cu at (112.4, 101.5)
- added C12: 0.1uF, Capacitors_SMD:C_0805_HandSoldering, B.Cu at (119.2, 121.0)
- added C13: 0.1uF, Capacitors_SMD:C_0805_HandSoldering, B.Cu at (157.9, 120.9)
- added C14: 0.1uF, Capacitors_SMD:C_0805_HandSoldering, B.Cu at (195.5, 120.8)
- added C15: 0.1uF, Capacitors_SMD:C_0805_HandSoldering, B.Cu at (195.7, 113.2)
- added C2: 0.1uF, Capacitors_SMD:C_0805_HandSoldering, B.Cu at (186.3, 100.5)
- added C3: 0.1uF, Capacitors_SMD:C_0805_HandSoldering, B.Cu at (178.1, 88.4)
- added C4: 4.7uF, Capacitors_SMD:C_0805_HandSoldering, B.Cu at (209.7, 81.3)
- added C5: 0.1uF, Capacitors_SMD:C_0805_HandSoldering, B.Cu at (178.1, 86.0)
- added C6: 1uF, Capacitors_SMD:C_0805_HandSoldering, B.Cu at (191.2, 76.5)
- added C7: 4.7uF, Capacitors_SMD:C_0805_HandSoldering, B.Cu at (176.1, 70.2)
- added C9: 0.1uF, Capacitors_SMD:C_0805_HandSoldering, B.Cu at (163.2, 83.2)
- added D1: D_ALT, Diodes_SMD:D_SOD-123, B.Cu at (207.5, 39.9)
- added D10: D_ALT, Diodes_SMD:D_SOD-123, B.Cu at (202.8, 39.9)
- added D11: D_ALT, Diodes_SMD:D_SOD-123, B.Cu at (235.4, 20.7)
- added D12: D_ALT, Diodes_SMD:D_SOD-123, B.Cu at (230.6, 18.3)
- added D13: D_ALT, Diodes_SMD:D_SOD-123, B.Cu at (212.3, 43.7)
- added D14: D_ALT, Diodes_SMD:D_SOD-123, B.Cu at (226.5, 41.8)
- added D15: D_ALT, Diodes_SMD:D_SOD-123, B.Cu at (230.6, 16.0)
- added D16: D_ALT, Diodes_SMD:D_SOD-123, B.Cu at (183.8, 41.3)
- added D17: D_ALT, Diodes_SMD:D_SOD-123, B.Cu at (169.5, 43.7)
- added D18: D_ALT, Diodes_SMD:D_SOD-123, B.Cu at (188.5, 43.7)
- added D19: D_ALT, Diodes_SMD:D_SOD-123, B.Cu at (235.4, 16.0)
- added D2: D_ALT, Diodes_SMD:D_SOD-123, B.Cu at (188.5, 41.3)
- added D20: D_ALT, Diodes_SMD:D_SOD-123, B.Cu at (235.4, 18.3)
- added D21: D_ALT, Diodes_SMD:D_SOD-123, B.Cu at (251.0, 14.9)
- added D22: D_ALT, Diodes_SMD:D_SOD-123, B.Cu at (251.0, 17.3)
- added D23: D_ALT, Diodes_SMD:D_SOD-123, B.Cu at (255.8, 19.6)
- added D24: D_ALT, Diodes_SMD:D_SOD-123, B.Cu at (251.0, 19.6)
- added D3: D_ALT, Diodes_SMD:D_SOD-123, B.Cu at (164.8, 43.7)
- added D4: D_ALT, Diodes_SMD:D_SOD-123, B.Cu at (183.8, 43.7)
- added D5: D_ALT, Diodes_SMD:D_SOD-123, B.Cu at (179.0, 41.3)
- added D6: D_ALT, Diodes_SMD:D_SOD-123, B.Cu at (179.0, 43.7)
- added D7: D_ALT, Diodes_SMD:D_SOD-123, B.Cu at (174.3, 39.9)
- added D8: D_ALT, Diodes_SMD:D_SOD-123, B.Cu at (221.8, 41.8)
- added D9: D_ALT, Diodes_SMD:D_SOD-123, B.Cu at (230.6, 20.7)
- added F1: 500mA Hold, Fuse_Holders_and_Fuses:Fuse_SMD1206_HandSoldering, B.Cu at (198.7, 69.9)
- added LED1: WS2812B, WS2812B:WS2812B, B.Cu at (167.4, 83.4)
- added LED2: WS2812B, WS2812B:WS2812B, B.Cu at (129.3, 83.6)
- added LED3: WS2812B, WS2812B:WS2812B, B.Cu at (112.3, 105.5)
- added LED4: WS2812B, WS2812B:WS2812B, B.Cu at (119.1, 125.1)
- added LED5: WS2812B, WS2812B:WS2812B, B.Cu at (157.9, 125.1)
- added LED6: WS2812B, WS2812B:WS2812B, B.Cu at (195.5, 125.2)
- added LED7: WS2812B, WS2812B:WS2812B, B.Cu at (195.8, 108.8)
- added MX1: MX-1U, MX_Alps_Hybrid:MX-1U, F.Cu at (100.7, 77.6)
- added MX10: MX-1U, MX_Alps_Hybrid:MX-1U, F.Cu at (162.6, 96.7)
- added MX11: MX-1U, MX_Alps_Hybrid:MX-1U, F.Cu at (181.7, 96.7)
- added MX12: MX-1.25U, MX_Alps_Hybrid:MX-1.25U, F.Cu at (203.1, 96.7)
- added MX13: MX-1U, MX_Alps_Hybrid:MX-1U, F.Cu at (110.2, 115.7)
- added MX14: MX-1U, MX_Alps_Hybrid:MX-1U, F.Cu at (129.2, 115.7)
- added MX15: MX-1U, MX_Alps_Hybrid:MX-1U, F.Cu at (148.3, 115.7)
- added MX16: MX-1U, MX_Alps_Hybrid:MX-1U, F.Cu at (167.4, 115.7)
- added MX17: MX-1U, MX_Alps_Hybrid:MX-1U, F.Cu at (186.4, 115.7)
- added MX18: MX-1U, MX_Alps_Hybrid:MX-1U, F.Cu at (205.5, 115.7)
- added MX19: MX-1U, MX_Alps_Hybrid:MX-1U, F.Cu at (105.4, 134.8)
- added MX2: MX-1U, MX_Alps_Hybrid:MX-1U, F.Cu at (119.7, 77.6)
- added MX20: MX-1.25U, MX_Alps_Hybrid:MX-1.25U, F.Cu at (126.9, 134.8)
- added MX21: MX-1U, MX_Alps_Hybrid:MX-1U, F.Cu at (148.3, 134.8)
- added MX22: MX-1U, MX_Alps_Hybrid:MX-1U, F.Cu at (167.4, 134.8)
- added MX23: MX-1U, MX_Alps_Hybrid:MX-1U, F.Cu at (186.4, 134.8)
- added MX24: MX-1U, MX_Alps_Hybrid:MX-1U, F.Cu at (205.5, 134.8)
- added MX25: MX-1.25U, MX_Alps_Hybrid:MX-1.25U, F.Cu at (203.1, 134.8)
- added MX26: MX-1.25U, MX_Alps_Hybrid:MX-1.25U, F.Cu at (179.3, 134.8)
- added MX27: MX-1.25U, MX_Alps_Hybrid:MX-1.25U, F.Cu at (155.5, 134.8)
- added MX28: MX-1U, MX_Alps_Hybrid:MX-1U, F.Cu at (134.1, 134.8)
- added MX29: MX-2.25U, MX_Alps_Hybrid:MX-2.25U, F.Cu at (117.4, 134.8)
- added MX3: MX-1U, MX_Alps_Hybrid:MX-1U, F.Cu at (138.8, 77.6)
- added MX30: MX-1.5U, MX_Alps_Hybrid:MX-1.5U, F.Cu at (110.2, 134.8)
- added MX4: MX-1U, MX_Alps_Hybrid:MX-1U, F.Cu at (157.9, 77.6)
- added MX5: MX-1U, MX_Alps_Hybrid:MX-1U, F.Cu at (176.9, 77.6)
- added MX6: MX-1.5U, MX_Alps_Hybrid:MX-1.5U, F.Cu at (200.7, 77.6)
- added MX7: MX-1U, MX_Alps_Hybrid:MX-1U, F.Cu at (105.4, 96.7)
- added MX8: MX-1U, MX_Alps_Hybrid:MX-1U, F.Cu at (124.5, 96.7)
- added MX9: MX-1U, MX_Alps_Hybrid:MX-1U, F.Cu at (143.6, 96.7)
- added NPNR1: 1.5k, Resistors_SMD:R_0805_HandSoldering, B.Cu at (172.0, 97.1)
- added Q1: Q_NPN_BCE, Keebio-Parts:SOT-23_Handsoldering, B.Cu at (172.2, 103.0)
- added R1: 10k, Resistors_SMD:R_0805_HandSoldering, B.Cu at (210.8, 97.1)
- added R10: R_Small, Resistors_SMD:R_0805_HandSoldering, B.Cu at (198.0, 40.2)
- added R11: R_Small, Resistors_SMD:R_0805_HandSoldering, B.Cu at (202.8, 43.9)
- added R12: R_Small, Resistors_SMD:R_0805_HandSoldering, B.Cu at (207.5, 43.9)
- added R13: R_Small, Resistors_SMD:R_0805_HandSoldering, B.Cu at (202.8, 42.0)
- added R14: R_Small, Resistors_SMD:R_0805_HandSoldering, B.Cu at (174.3, 42.0)
- added R15: R_Small, Resistors_SMD:R_0805_HandSoldering, B.Cu at (174.3, 43.9)
- added R16: R_Small, Resistors_SMD:R_0805_HandSoldering, B.Cu at (169.5, 39.7)
- added R17: R_Small, Resistors_SMD:R_0805_HandSoldering, B.Cu at (169.5, 41.6)
- added R18: R_Small, Resistors_SMD:R_0805_HandSoldering, B.Cu at (164.8, 39.7)
- added R19: R_Small, Resistors_SMD:R_0805_HandSoldering, B.Cu at (164.8, 41.6)
- added R2: 10k, Resistors_SMD:R_0805_HandSoldering, B.Cu at (204.6, 86.0)
- added R20: R_Small, Resistors_SMD:R_0805_HandSoldering, B.Cu at (226.5, 43.9)
- added R21: R_Small, Resistors_SMD:R_0805_HandSoldering, B.Cu at (221.8, 43.9)
- added R22: R_Small, Resistors_SMD:R_0805_HandSoldering, B.Cu at (217.0, 40.2)
- added R23: R_Small, Resistors_SMD:R_0805_HandSoldering, B.Cu at (217.0, 42.0)
- added R24: R_Small, Resistors_SMD:R_0805_HandSoldering, B.Cu at (217.0, 43.9)
- added R25: R_Small, Resistors_SMD:R_0805_HandSoldering, B.Cu at (212.3, 39.7)
- added R26: R_Small, Resistors_SMD:R_0805_HandSoldering, B.Cu at (212.3, 41.6)
- added R27: R_Small, Resistors_SMD:R_0805_HandSoldering, B.Cu at (221.8, 39.7)
- added R28: R_Small, Resistors_SMD:R_0805_HandSoldering, B.Cu at (207.5, 42.0)
- added R3: 4.7k, Resistors_SMD:R_0805_HandSoldering, B.Cu at (110.1, 87.9)
- added R4: 4.7k, Resistors_SMD:R_0805_HandSoldering, B.Cu at (110.1, 85.9)
- added R5: R_Small, Resistors_SMD:R_0805_HandSoldering, B.Cu at (193.3, 43.9)
- added R6: R_Small, Resistors_SMD:R_0805_HandSoldering, B.Cu at (193.3, 42.0)
- added R7: R_Small, Resistors_SMD:R_0805_HandSoldering, B.Cu at (193.3, 40.2)
- added R8: R_Small, Resistors_SMD:R_0805_HandSoldering, B.Cu at (198.0, 43.9)
- added R9: R_Small, Resistors_SMD:R_0805_HandSoldering, B.Cu at (198.0, 42.0)
- added RGBR1: 470, Resistors_SMD:R_0805_HandSoldering, B.Cu at (171.8, 83.0)
- added SPI1: 2x3 SPI, Pin_Headers:Pin_Header_Straight_2x03_Pitch2.00mm, B.Cu at (210.9, 91.4)
- added TRRS1: TRRS1, Keebio-Parts:TRRS-PJ-320A, B.Cu at (110.2, 67.3)
- added U1: ATmega32U4, keyboard_parts:QFP44, B.Cu at (191.1, 86.0)
- added U2: PRTR5V0U2X, Nexperia:SOT143B, B.Cu at (210.7, 70.5)
- added UR1: 22, Resistors_SMD:R_0805_HandSoldering, B.Cu at (209.8, 74.6)
- added UR2: 22, Resistors_SMD:R_0805_HandSoldering, B.Cu at (211.7, 74.7)
- added UR3: 5.1k, Resistors_SMD:R_0805_HandSoldering, B.Cu at (168.1, 72.1)
- added UR4: 5.1k, Resistors_SMD:R_0805_HandSoldering, B.Cu at (166.5, 70.2)
- added UR5: 1M, Resistors_SMD:R_0805_HandSoldering, B.Cu at (171.4, 70.2)
- added USB1: HRO-TYPE-C-31-M-12, Type-C:HRO-TYPE-C-31-M-12-HandSoldering, B.Cu at (189.4, 65.0)
- added XC1: 22pF, Capacitors_SMD:C_0805_HandSoldering, B.Cu at (189.9, 100.5)
- added XC2: 22pF, Capacitors_SMD:C_0805_HandSoldering, B.Cu at (197.9, 100.5)
- added Y1: Crystal_GND2, keyboard_parts:Crystal_SMD_3225-4pin_3.2x2.5mm, B.Cu at (194.0, 100.7)
- SW1: footprint Cherry_MX_Matias_u1_NoSilk_Back -> Buttons_Switches_SMD:SW_SPST_SKQG; moved to B.Cu
- moved SW1 113.0 mm to (210.5, 104.1), turned to 90 degrees
Routing:
- net Net-(U1-Pad17): track 0.00 -> 13.4 mm
- net Net-(U1-Pad16): track 0.00 -> 11.6 mm
- net Net-(U2-Pad3): track 0.00 -> 3.90 mm
- net Net-(U2-Pad2): track 0.00 -> 3.90 mm
- added copper zone on B.Cu, net GND
- added copper zone on F.Cu, net GND
Other:
- board size 128.5 x 81 mm -> 124.1 x 77.9 mm
- net class Default: clearance 0.2 -> 0.1524; trace_width 0.25 -> 0.204; via_dia 0.8 -> 0.6
- net class POWER added: clearance 0.1524, trace_width 0.381, via_dia 0.6, via_drill 0.4
- rule trace_clearance: 0.2 -> 0.1524
