File: TS48_Right/TS48_right.sch (KiCad schematic (older format))
At the start: 43 parts, among them Q1 Q_NPN_BCE, SW1 SW_PUSH, U1 ATmega32U4, U2 PRTR5V0U2X, Y1 Crystal_GND2

Commit message: Layout changes
Parts:
- SPI1: footprint keyboard_parts:Pin_Header_Straight_2x03_Pitch1.27mm -> Pin_Headers:Pin_Header_Straight_2x03_Pitch2.00mm
Changed lines of the file:
@@
 F 0 "SPI1" H 21250 10200 50  0000 C CNN
 F 1 "2x3 SPI" H 21250 9800 50  0000 C CNN
-F 2 "keyboard_parts:Pin_Header_Straight_2x03_Pitch1.27mm" H 21200 10000 50  0001 C CNN
+F 2 "Pin_Headers:Pin_Header_Straight_2x03_Pitch2.00mm" H 21200 10000 50  0001 C CNN
 F 3 "" H 21200 10000 50  0001 C CNN
 	1    21200 10000
@@
 L power:GND #PWR020
 U 1 1 5B54C788
-P 19375 14375
-F 0 "#PWR020" H 19375 14125 50  0001 C CNN
-F 1 "GND" H 19375 14225 50  0000 C CNN
-F 2 "" H 19375 14375 50  0001 C CNN
-F 3 "" H 19375 14375 50  0001 C CNN
-	1    19375 14375
+P 19350 14375
+F 0 "#PWR020" H 19350 14125 50  0001 C CNN
+F 1 "GND" H 19350 14225 50  0000 C CNN
+F 2 "" H 19350 14375 50  0001 C CNN
+F 3 "" H 19350 14375 50  0001 C CNN
+	1    19350 14375
 	1    0    0    -1
 $EndComp

Commit message: Routing
Connections:
- net labels added: COL0, COL1, COL2, COL3, COL4, COL5, ROW0, ROW1, ROW2, ROW3
- wire segments 217 -> 218
Other:
- moved on the sheet: C4
Changed lines of the file:
@@
 L device:C_Small C4
 U 1 1 5B4A929A
-P 16925 10725
-F 0 "C4" H 16935 10795 50  0000 L CNN
-F 1 "4.7uF" H 16935 10645 50  0000 L CNN
-F 2 "Capacitors_SMD:C_0805_HandSoldering" H 16925 10725 50  0001 C CNN
-F 3 "" H 16925 10725 50  0001 C CNN
-	1    16925 10725
+P 17000 10775
+F 0 "C4" H 17010 10845 50  0000 L CNN
+F 1 "4.7uF" H 17010 10695 50  0000 L CNN
+F 2 "Capacitors_SMD:C_0805_HandSoldering" H 17000 10775 50  0001 C CNN
+F 3 "" H 17000 10775 50  0001 C CNN
+	1    17000 10775
 	1    0    0    -1
 $EndComp
@@
 	17400 10625 17400 10725
 Connection ~ 19775 10625
-Wire Wire Line
-	17400 10625 16925 10625
 Connection ~ 17400 10625
 Connection ~ 17400 10725
@@
 Wire Wire Line
 	17400 11025 17400 10925
-Wire Wire Line
-	17400 10925 16925 10925
-Wire Wire Line
-	16925 10925 16925 10825
 Connection ~ 17400 10925
-Wire Wire Line
-	16925 10625 16700 10625
-Connection ~ 16925 10625
-Wire Wire Line
-	16925 10925 16700 10925
-Connection ~ 16925 10925
 Wire Wire Line
 	20025 12625 19025 12625
@@
 	1    0    0    -1
 $EndComp
+Text GLabel 22575 10625 2    50   Input ~ 0
+COL5
+Text GLabel 22575 11025 2    50   Input ~ 0
+COL1
+Text GLabel 22575 11525 2    50   Input ~ 0
+COL0
+Text GLabel 22575 12025 2    50   Input ~ 0
+ROW3
+Text GLabel 22575 12125 2    50   Input ~ 0
+ROW2
+Text GLabel 22575 12225 2    50   Input ~ 0
+COL4
+Text GLabel 22575 12325 2    50   Input ~ 0
+ROW1
+Text GLabel 22575 12425 2    50   Input ~ 0
+COL3
+Text GLabel 22575 12525 2    50   Input ~ 0
+COL2
+Text GLabel 22600 13025 2    50   Input ~ 0
+ROW0
+Wire Wire Line
+	16700 10925 17000 10925
+Wire Wire Line
+	16700 10625 17000 10625
+Wire Wire Line
+	17000 10875 17000 10925
+Connection ~ 17000 10925
+Wire Wire Line
+	17000 10925 17400 10925
+Wire Wire Line
+	17000 10675 17000 10625
+Connection ~ 17000 10625
+Wire Wire Line
+	17000 10625 17400 10625
 $EndSCHEMATC

Commit message: Routed board
Changed lines of the file:
@@
 Wire Wire Line
 	24500 12700 24500 11850
-Wire Wire Line
-	25050 12700 25050 12800
-Connection ~ 25050 12800
 $Comp
 L power:GND #PWR0101
@@
 Wire Wire Line
 	24075 12750 24025 12750
-Connection ~ 24075 12750
 Wire Wire Line
 	24375 12925 25050 12925
-Wire Wire Line
-	25050 12800 25050 12925
 Connection ~ 24375 12925
 Wire Wire Line
@@
 Connection ~ 25050 12925
 Wire Wire Line
-	25050 12700 25050 12275
-Wire Wire Line
 	25050 12275 24650 12275
-Connection ~ 25050 12700
 Connection ~ 24650 12275
 Wire Wire Line
@@
 Wire Wire Line
 	17000 10625 17400 10625
+Wire Wire Line
+	25050 12275 25050 12700
+Connection ~ 25050 12700
+Wire Wire Line
+	25050 12700 25050 12800
+Connection ~ 25050 12800
+Wire Wire Line
+	25050 12800 25050 12925
+Connection ~ 24075 12750
 $EndSCHEMATC

Commit message: cLEANUP
Parts:
- SPI1: symbol conn:Conn_02x03_Odd_Even -> TS48_right-rescue:Conn_02x03_Odd_Even-conn
- TRRS1: symbol conn:Audio-Jack-4 -> TS48_right-rescue:Audio-Jack-4-conn
- U1: symbol atmel:ATmega32U4 -> TS48_right-rescue:ATmega32U4-atmel
Changed lines of the file:
@@
 EESchema Schematic File Version 4
 LIBS:TS48_right-cache
-EELAYER 26 0
+EELAYER 29 0
 EELAYER END
 $Descr A0 46811 33110
@@
 D-
 $Comp
-L atmel:ATmega32U4 U1
+L TS48_right-rescue:ATmega32U4-atmel U1
 U 1 1 5B4A9FC2
 P 21275 12175
@@
 RGBIN
 $Comp
-L conn:Conn_02x03_Odd_Even SPI1
+L TS48_right-rescue:Conn_02x03_Odd_Even-conn SPI1
 U 1 1 5B544D39
 P 21200 10000
@@
 $EndComp
 $Comp
-L conn:Audio-Jack-4 TRRS1
+L TS48_right-rescue:Audio-Jack-4-conn TRRS1
 U 1 1 5B94F9A5
 P 25625 10875
