File: TS48_left/TS48_left.kicad_pcb (KiCad board)
At the start: 2 copper layers, 124 x 77.9 mm, 121 parts, among them Q1 Q_NPN_BCE, SW1 SW_PUSH, U1 ATmega32U4, U2 PRTR5V0U2X, Y1 

Commit message: Optimising routing
Routing:
- net COL0: track 70.3 -> 105.8 mm, vias 1 -> 3
- net +5V: track 727.8 -> 742.4 mm
- net ROW0: track 172.3 -> 177.3 mm
- net GND: track 75.2 -> 78.2 mm, vias 87 -> 94
- net Net-(D13-Pad2): track 11.6 -> 12.7 mm
- net SCK: track 31.8 -> 32.6 mm
- net D+: track 30.7 -> 31.3 mm
Other:
- board text added: "REV 1.0"
- board text removed: "REV 1"
