File: TS48_left/TS48_left.sch (KiCad schematic (older format))
At the start: 43 parts, among them Q1 Q_NPN_BCE, SW1 SW_PUSH, U1 ATmega32U4, U2 PRTR5V0U2X, Y1 Crystal_GND2

Commit message: BOM
Parts:
- SPI1: symbol conn:Conn_02x03_Odd_Even -> TS48_left-rescue:Conn_02x03_Odd_Even-conn
- TRRS1: symbol conn:Audio-Jack-4 -> TS48_left-rescue:Audio-Jack-4-conn
- U1: symbol atmel:ATmega32U4 -> TS48_left-rescue:ATmega32U4-atmel
Changed lines of the file:
@@
 EESchema Schematic File Version 4
 LIBS:TS48_left-cache
-EELAYER 26 0
+EELAYER 29 0
 EELAYER END
 $Descr A4 11693 8268
@@
 D-
 $Comp
-L atmel:ATmega32U4 U1
+L TS48_left-rescue:ATmega32U4-atmel U1
 U 1 1 5B4A9FC2
 P 5600 3175
@@
 RGBIN
 $Comp
-L conn:Conn_02x03_Odd_Even SPI1
+L TS48_left-rescue:Conn_02x03_Odd_Even-conn SPI1
 U 1 1 5B544D39
 P 5525 1000
@@
 $EndComp
 $Comp
-L conn:Audio-Jack-4 TRRS1
+L TS48_left-rescue:Audio-Jack-4-conn TRRS1
 U 1 1 5B94F9A5
 P 9950 1875
